File: lfo.kicad_pcb (KiCad board)
At the start: 2 copper layers, 30 x 234.4 mm, 95 parts, among them J1 Conn_02x05_Odd_Even, J2 AudioJack2_SwitchT, J3 AudioJack2_SwitchT, J4 AudioJack2_SwitchT, J5 AudioJack2_SwitchT, J6 AudioJack2_SwitchT, J7 AudioJack2_SwitchT, Q1 BC557, Q2 BS170, Q3 BC547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

Commit message: fix pcb
Parts:
- C9: footprint Capacitor_SMD:C_0805_2012Metric -> Capacitor_SMD:C_0603_1608Metric_Pad1.08x0.95mm_HandSolder
Changed lines of the file:
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@@
     )
   )
-  (footprint "Capacitor_SMD:C_0805_2012Metric" (layer "B.Cu")
+  (footprint "Capacitor_SMD:C_0603_1608Metric_Pad1.08x0.95mm_HandSolder" (layer "B.Cu")
     (at 86.106 95.486 180)
-    (descr "Capacitor SMD 0805 (2012 Metric), square (rectangular) end terminal, IPC_7351 nominal, (Body size source: IPC-SM-782 page 76, https://www.pcb-3d.com/wordpress/wp-content/uploads/ipc-sm-782a_amendment_1_and_2.pdf, https://docs.google.com/spreadsheets/d/1BsfQQcO9C6DZCsRaXUlFlo91Tg2WpOkGARC1WS5S8t0/edit?usp=sharing), generated with kicad-footprint-generator")
-    (tags "capacitor")
+    (descr "Capacitor SMD 0603 (1608 Metric), square (rectangular) end terminal, IPC_7351 nominal with elongated pad for handsoldering. (Body size source: IPC-SM-782 page 76, https://www.pcb-3d.com/wordpress/wp-content/uploads/ipc-sm-782a_amendment_1_and_2.pdf), generated with kicad-footprint-generator")
+    (tags "capacitor handsolder")
     (property "Sheetfile" "lfo.kicad_sch")
     (property "Sheetname" "")
@@
     (property "ki_keywords" "cap capacitor")
     (attr smd)
-    (fp_text reference "C9" (at 3.048 -0.127) (layer "B.SilkS")
+    (fp_text reference "C9" (at 2.794 -0.018) (layer "B.SilkS")
         (effects (font (size 1 1) (thickness 0.15)) (justify mirror))
     )
-    (fp_text value "120p" (at 0 -1.68) (layer "B.Fab")
+    (fp_text value "120p" (at 0 -1.43) (layer "B.Fab")
         (effects (font (size 1 1) (thickness 0.15)) (justify mirror))
     )
     (fp_text user "${REFERENCE}" (at 0 0) (layer "B.Fab")
-        (effects (font (size 0.5 0.5) (thickness 0.08)) (justify mirror))
+        (effects (font (size 0.4 0.4) (thickness 0.06)) (justify mirror))
     )
-    (fp_line (start -0.261252 -0.735) (end 0.261252 -0.735)
+    (fp_line (start -0.146267 -0.51) (end 0.146267 -0.51)
       (stroke (width 0.12) (type solid)) (layer "B.SilkS"))
-    (fp_line (start -0.261252 0.735) (end 0.261252 0.735)
+    (fp_line (start -0.146267 0.51) (end 0.146267 0.51)
       (stroke (width 0.12) (type solid)) (layer "B.SilkS"))
-    (fp_line (start -1.7 -0.98) (end -1.7 0.98)
+    (fp_line (start -1.65 -0.73) (end -1.65 0.73)
       (stroke (width 0.05) (type solid)) (layer "B.CrtYd"))
-    (fp_line (start -1.7 0.98) (end 1.7 0.98)
+    (fp_line (start -1.65 0.73) (end 1.65 0.73)
       (stroke (width 0.05) (type solid)) (layer "B.CrtYd"))
-    (fp_line (start 1.7 -0.98) (end -1.7 -0.98)
+    (fp_line (start 1.65 -0.73) (end -1.65 -0.73)
       (stroke (width 0.05) (type solid)) (layer "B.CrtYd"))
-    (fp_line (start 1.7 0.98) (end 1.7 -0.98)
+    (fp_line (start 1.65 0.73) (end 1.65 -0.73)
       (stroke (width 0.05) (type solid)) (layer "B.CrtYd"))
-    (fp_line (start -1 -0.625) (end -1 0.625)
+    (fp_line (start -0.8 -0.4) (end -0.8 0.4)
       (stroke (width 0.1) (type solid)) (layer "B.Fab"))
-    (fp_line (start -1 0.625) (end 1 0.625)
+    (fp_line (start -0.8 0.4) (end 0.8 0.4)
       (stroke (width 0.1) (type solid)) (layer "B.Fab"))
-    (fp_line (start 1 -0.625) (end -1 -0.625)
+    (fp_line (start 0.8 -0.4) (end -0.8 -0.4)
       (stroke (width 0.1) (type solid)) (layer "B.Fab"))
-    (fp_line (start 1 0.625) (end 1 -0.625)
+    (fp_line (start 0.8 0.4) (end 0.8 -0.4)
       (stroke (width 0.1) (type solid)) (layer "B.Fab"))
-    (pad "1" smd roundrect (at -0.95 0 180) (size 1 1.45) (layers "B.Cu" "B.Paste" "B.Mask") (roundrect_rratio 0.25)
+    (pad "1" smd roundrect (at -0.8625 0 180) (size 1.075 0.95) (layers "B.Cu" "B.Paste" "B.Mask") (roundrect_rratio 0.25)
       (net 47 "Net-(U3A--)") (pintype "passive"))
-    (pad "2" smd roundrect (at 0.95 0 180) (size 1 1.45) (layers "B.Cu" "B.Paste" "B.Mask") (roundrect_rratio 0.25)
+    (pad "2" smd roundrect (at 0.8625 0 180) (size 1.075 0.95) (layers "B.Cu" "B.Paste" "B.Mask") (roundrect_rratio 0.25)
       (net 11 "Net-(C9-Pad2)") (pintype "passive"))
-    (model "${KICAD6_3DMODEL_DIR}/Capacitor_SMD.3dshapes/C_0805_2012Metric.wrl"
+    (model "${KICAD6_3DMODEL_DIR}/Capacitor_SMD.3dshapes/C_0603_1608Metric.wrl"
       (offset (xyz 0 0 0))
       (scale (xyz 1 1 1))

Commit message: annotating some issues
Routing:
- net GND: track 76.6 -> 111.6 mm, vias 4 -> 6
- net Net-(R24-Pad2): track 24.0 -> 33.2 mm
- net +12V: track 188.1 -> 193.2 mm
- net Net-(Q1-C): track 107.1 -> 104.9 mm
- net Net-(Q2-G): track 13.8 -> 15.1 mm
- net Net-(D2-A): track 25.3 -> 26.0 mm
- net Net-(SW1B-C): track 15.0 -> 15.6 mm
- net Net-(Q1-B): track 12.9 -> 12.3 mm
- net Net-(R11-Pad2): track 30.9 -> 31.5 mm
